File: pill-dispenser.kicad_sch (KiCad schematic)
At the start: 34 parts, among them J1 USB-C, J3 WS2812B, J4 Button, J5 Wakeup Button, Q1 AO3401A, Q2 FS8205A, SW1 Battery Switch, U1 MT3608, U2 ESP32-C3-Zero, U3 TP4056-42-ESOP8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

Commit message: Added control led strip transotor, placed buttons on PCB
Parts:
- removed J4: Button, Connector_PinSocket_2.54mm:PinSocket_1x02_P2.54mm_Horizontal, symbol Connector_Generic:Conn_01x02
- removed J5: Wakeup Button, Connector_PinSocket_2.54mm:PinSocket_1x02_P2.54mm_Horizontal, symbol Connector_Generic:Conn_01x02
- added S1: Reset Button, FSMRA6JH:SW_FSMRA6JH, symbol FSMRA6JH:FSMRA6JH
- added S2: Button, FSMRA6JH:SW_FSMRA6JH, symbol FSMRA6JH:FSMRA6JH
- added U5: IRLML2502, IRLML2502TRPBF:SOT23, symbol IRLML2502TRPBF:IRLML2502TRPBF
- BZ1: CHIPDIP https://www.chipdip.ru/product0/8307188362 -> https://www.chipdip.ru/product0/9001617446
Connections:
- net BUTTON: now also S2.1
- net GND: now also S1.2, S2.2, U5.2; no longer J3.1 (Pin_1)
- net WAKEUP_BUT: now also S1.1
- net at C4.2, Q2.2, Q2.3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: now also BT1.2 (-); no longer SW1.5
- net at SW1.6: no longer BT1.2 (-)
- net LED_STRIP_ENABLE: now reaches U2.8 (IO4)
- net LED_STRIP_ENABLE: now also U5.1
- net LED_STRIP renamed LED_STRIP_CONTROL
- new net: S2.S1 (SHIELD), S2.S2 (SHIELD)
- new net: J3.1 (Pin_1), U5.3
- new net: S1.S1 (SHIELD), S1.S2 (SHIELD)
- no-connect marks 20 -> 23
Other:
- moved on the sheet: BZ1, J3
